File: Eagle/DMTV_SD.brd (EAGLE design)
At the start: 78.6 x 55.7 mm, 71 parts, among them J1 181-015-213R561, J2 2-1735446-7, J4 35RASMT2BHNTRX, U1 ICE40HX1K-VQ100, U2 SN74LVC245APWR, U3 MCU-ATMEGA32U4-MUR(VQFN44), Y1 16MHz

Commit message: Signed-off-by: GameboxSystems <gamebox.systems@gmail.com>
Connections:
- new net BTNA: U1.82, U2.13
- new net BTNB: U1.86, U2.14
- net D10: no longer U1.87
- net D11: now also U2.7; no longer U1.82
- net D7: no longer U1.83
- net D8: no longer U1.85
- net D9: now also U2.6; no longer U1.86
- net GND: no longer U2.6, U2.7
Routing:
- net D8: track 41.3 -> 0.00 mm, vias 2 -> 0
- net D10: track 39.5 -> 0.00 mm
- net D7: track 30.2 -> 0.00 mm, vias 2 -> 0
- net BTNA: track 0.00 -> 21.1 mm, vias 0 -> 2
- net BTNB: track 0.00 -> 19.9 mm, vias 0 -> 2
- net D11: track 35.8 -> 31.4 mm
- net D9: track 39.8 -> 38.4 mm
- net D6: track 20.0 -> 19.4 mm
